Commit message: add_new_multiple_envs

File: ManiSkill2_real2sim/mani_skill2_real2sim/assets/descriptions/googlerobot_description/google_robot_meta_sim_fix_wheel_fix_fingertip.urdf (robot description, URDF)
Before this commit: robot meta, 37 links, 36 joints
Links:
- link link_finger_tip_left: geometry collision mesh filename=coarse_meshes/link_finger_tip_boxified.obj; visual mesh filename=3obj/link_finger_tip_simplified.3obj.obj
- link link_finger_tip_right: geometry collision mesh filename=coarse_meshes/link_finger_tip_boxified.obj; visual mesh filename=3obj/link_finger_tip_simplified.3obj.obj
